File: boards/handheld_tracker/handheld_tracker.kicad_sch (KiCad schematic)
At the start: 15 parts, among them U1 SAM-M8Q, U2 RFM96W-433S2, U4 LM3670MF

Commit message: added all footprints and modified gitignore
Parts:
- AE1: footprint (none) -> Connector_Coaxial:SMA_Amphenol_901-143_Horizontal
- C4, C5: footprint (none) -> Capacitor_SMD:C_0805_2012Metric
- L1: footprint (none) -> Inductor_SMD:L_0805_2012Metric
Other:
- sheet mcu ports: added display_RST; removed display_CS
- sheet user_interface ports: added I2C_SCL, I2C_SDA, display_RST; removed MISO, MOSI, SCK, display_CS
Changed lines of the file:
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@@
+		)
+	)
+	(label "I2C_SCL"
+		(at 162.56 128.27 0)
+		(fields_autoplaced yes)
+		(effects
+			(font
+				(size 1.27 1.27)
+			)
+			(justify left bottom)
 		)
 	)
@@
 		)
 	)
+	(label "display_RST"
+		(at 68.58 54.61 0)
+		(fields_autoplaced yes)
+		(effects
+			(font
+				(size 1.27 1.27)
+			)
+			(justify left bottom)
+		)
+	)
 	(label "pushbutton_8"
 		(at 31.75 53.34 180)
@@
 		)
 	)
+	(label "display_RST"
+		(at 162.56 134.62 0)
+		(fields_autoplaced yes)
+		(effects
+			(font
+				(size 1.27 1.27)
+			)
+			(justify left bottom)
+		)
+	)
 	(label "pushbutton_1"
 		(at 123.19 119.38 180)
@@
 	)
 	(label "I2C_SCL"
-		(at 68.58 60.96 0)
+		(at 68.58 64.77 0)
 		(fields_autoplaced yes)
 		(effects
@@
 		)
 	)
+	(label "I2C_SDA"
+		(at 162.56 130.81 0)
+		(fields_autoplaced yes)
+		(effects
+			(font
+				(size 1.27 1.27)
+			)
+			(justify left bottom)
+		)
+	)
 	(label "SCK"
 		(at 198.12 111.76 180)
@@
 	)
 	(label "I2C_SDA"
-		(at 68.58 63.5 0)
+		(at 68.58 67.31 0)
 		(fields_autoplaced yes)
 		(effects
@@
 			)
 		)
-		(property "Footprint" ""
+		(property "Footprint" "Capacitor_SMD:C_0805_2012Metric"
 			(at 31.4452 144.78 0)
 			(effects
@@
 			)
 		)
-		(property "Footprint" ""
+		(property "Footprint" "Capacitor_SMD:C_0805_2012Metric"
 			(at 77.1652 144.78 0)
 			(effects
@@
 			)
 		)
-		(property "Footprint" ""
+		(property "Footprint" "Connector_Coaxial:SMA_Amphenol_901-143_Horizontal"
 			(at 236.22 44.45 0)
 			(effects
@@
 			)
 		)
-		(property "Footprint" ""
+		(property "Footprint" "Inductor_SMD:L_0805_2012Metric"
 			(at 63.5 137.16 0)
 			(effects
@@
 			)
 		)
-		(pin "display_CS" output
-			(at 68.58 52.07 0)
-			(effects
-				(font
-					(size 1.27 1.27)
-				)
-				(justify right)
-			)
-		)
 		(pin "transceiver_CS" output
-			(at 68.58 54.61 0)
+			(at 68.58 59.69 0)
 			(effects
 				(font
@@
 		)
 		(pin "I2C_SCL" output
-			(at 68.58 60.96 0)
+			(at 68.58 64.77 0)
 			(effects
 				(font
@@
 		)
 		(pin "I2C_SDA" bidirectional
-			(at 68.58 63.5 0)
+			(at 68.58 67.31 0)
 			(effects
 				(font
@@
 				)
 				(justify left)
+			)
+		)
+		(pin "display_RST" output
+			(at 68.58 54.61 0)
+			(effects
+				(font
+					(size 1.27 1.27)
+				)
+				(justify right)
 			)
 		)
@@
 			)
 		)
-		(pin "SCK" output
-			(at 162.56 124.46 0)
+		(pin "display_RST" input
+			(at 162.56 134.62 0)
 			(effects
 				(font
@@
 			)
 		)
-		(pin "MOSI" output
-			(at 162.56 127 0)
+		(pin "I2C_SDA" bidirectional
+			(at 162.56 130.81 0)
 			(effects
 				(font
@@
 			)
 		)
-		(pin "MISO" input
-			(at 162.56 129.54 0)
-			(effects
-				(font
-					(size 1.27 1.27)
-				)
-				(justify right)
-			)
-		)
-		(pin "display_CS" output
-			(at 162.56 132.08 0)
-			(effects
-				(font
+		(pin "I2C_SCL" input
+			(at 162.56 128.27 0)
+			(effects
+				(font

Commit message: basic pcb layout
Parts:
- renumbered TP6 to TP_3V3, TP7 to TP_GND1, TP4 to TP_I2C_SCL1, TP5 to TP_I2C_SDA1, TP8 to TP_INPUT_VOLTAGE1, TP2 to TP_MISO1, TP3 to TP_MOSI1, TP1 to TP_SCK1
Connections:
- net I2C_SCL: now also U1.12 (SCL)
- net I2C_SDA: now also U1.9 (SDA)
Other:
- moved on the sheet: TP_3V3, TP_GND1, TP_INPUT_VOLTAGE1
