File: boards/handheld_tracker/handheld_tracker.kicad_pcb (KiCad board)
At the start: 2 copper layers, 64 x 100 mm, 41 parts, among them J1 Conn_01x08_Pin, J2 Conn_01x02_Pin, SW0 SW_Push, SW1 SW_Push, SW2 SW_Push, SW3 SW_Push, SW4 SW_Push, SW5 SW_Push, SW6 SW_Push, SW7 SW_Push, SW8 SW_Push, SW9 SW_Push, U1 SAM-M8Q, U2 RFM96W-433S2, U3 ATmega328PB-A, U4 LM3670MF, Y1 Crystal

Commit message: finished board pre-review
Parts:
- removed TP_3V3, TP_GND1, TP_I2C_SCL1, TP_I2C_SDA1, TP_INPUT_VOLTAGE1, TP_MISO1, TP_MOSI1, TP_SCK1: TestPoint, TestPoint:TestPoint_Pad_D3.0mm
- added J3: Conn_01x02_Pin, Connector_PinHeader_2.54mm:PinHeader_1x02_P2.54mm_Vertical, F.Cu at (139.5, 49.0)
- added J4: Conn_01x05_Pin, Connector_PinHeader_2.54mm:PinHeader_1x05_P2.54mm_Vertical, F.Cu at (109.5, 59.1)
- added J5: Conn_01x03_Pin, Connector_PinHeader_2.54mm:PinHeader_1x03_P2.54mm_Vertical, F.Cu at (139.5, 56.0)
- moved C4 4.99 mm to (144.7, 62.5)
- moved C5 4.99 mm to (139.3, 63.5)
- moved L1 4.99 mm to (144.8, 72.5)
- moved U4 4.99 mm to (144.6, 67.5)
Connections:
- SW0 pad 1: +3.3V -> GND
- SW1 pad 1: +3.3V -> GND
- SW2 pad 1: +3.3V -> GND
- SW3 pad 1: +3.3V -> GND
- SW4 pad 1: +3.3V -> GND
- SW5 pad 1: +3.3V -> GND
- SW6 pad 1: +3.3V -> GND
- SW7 pad 1: +3.3V -> GND
- SW8 pad 1: +3.3V -> GND
- SW9 pad 1: +3.3V -> GND
- SW_DOT1 pad 1: +3.3V -> GND
- SW_DOWN1 pad 1: +3.3V -> GND
- SW_ENTER1 pad 1: +3.3V -> GND
- SW_MENU1 pad 1: +3.3V -> GND
- SW_UP1 pad 1: +3.3V -> GND
Routing:
- net /SCK: track 18.7 -> 88.0 mm
- net /MOSI: track 18.8 -> 84.7 mm, vias 0 -> 1
- net /MISO: track 20.6 -> 83.1 mm
- net /I2C_SDA: track 28.6 -> 74.0 mm, vias 0 -> 3
- net +3.3V: track 17.9 -> 59.0 mm, vias 3 -> 8
- net /I2C_SCL: track 18.9 -> 59.3 mm, vias 0 -> 3
- net /display_RST: track 0.00 -> 30.1 mm
- net INPUT_VOLTAGE: track 3.91 -> 20.0 mm
- net GND: track 9.04 -> 24.1 mm, vias 0 -> 1
- net Net-(R3-Pad2): track 4.54 -> 12.5 mm
- net /pushbutton_menu: track 22.0 -> 28.0 mm
- net /pushbutton_3: track 17.9 -> 23.9 mm
- net /pushbutton_2: track 27.2 -> 33.1 mm
- net /pushbutton_1: track 48.8 -> 54.8 mm
- net /pushbutton_up: track 35.1 -> 40.1 mm
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