File: boards/handheld_tracker/handheld_tracker.kicad_pcb (KiCad board)
At the start: 2 copper layers, 64 x 100 mm, 36 parts, among them J1 Conn_01x08_Pin, J2 Conn_01x02_Pin, J3 Conn_01x02_Pin, J4 Conn_01x05_Pin, J5 Conn_01x03_Pin, SW0 SW_Push, SW1 SW_Push, SW2 SW_Push, SW3 SW_Push, SW4 SW_Push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

Commit message: finished beacon schematic
Changed lines of the file:
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@@
 			(plot_on_all_layers_selection 0x0000000_00000000)
 			(disableapertmacros no)
-			(usegerberextensions no)
+			(usegerberextensions yes)
 			(usegerberattributes yes)
 			(usegerberadvancedattributes yes)
@@
 			(outputformat 1)
 			(mirror no)
-			(drillshape 1)
+			(drillshape 0)
 			(scaleselection 1)
-			(outputdirectory "")
+			(outputdirectory "gerbers/")
 		)
 	)
@@
 			(size 1.025 1.4)
 			(layers "F.Cu" "F.Paste" "F.Mask")
-			(roundrect_rratio 0.243902)
+			(roundrect_rratio 0.243902439)
 			(net 26 "/mcu/TX")
 			(pintype "passive")
@@
 			(size 1.025 1.4)
 			(layers "F.Cu" "F.Paste" "F.Mask")
-			(roundrect_rratio 0.243902)
+			(roundrect_rratio 0.243902439)
 			(net 51 "Net-(J2-Pin_1)")
 			(pintype "passive")
@@
 			(size 1.025 1.4)
 			(layers "F.Cu" "F.Paste" "F.Mask")
-			(roundrect_rratio 0.243902)
+			(roundrect_rratio 0.243902439)
 			(net 23 "/mcu/RX")
 			(pintype "passive")
@@
 			(size 1.025 1.4)
 			(layers "F.Cu" "F.Paste" "F.Mask")
-			(roundrect_rratio 0.243902)
+			(roundrect_rratio 0.243902439)
 			(net 52 "Net-(J2-Pin_2)")
 			(pintype "passive")
@@
 			(size 1.025 1.4)
 			(layers "F.Cu" "F.Paste" "F.Mask")
-			(roundrect_rratio 0.243902)
+			(roundrect_rratio 0.243902439)
 			(net 24 "/mcu/RESET")
 			(pintype "passive")
@@
 			(size 1.025 1.4)
 			(layers "F.Cu" "F.Paste" "F.Mask")
-			(roundrect_rratio 0.243902)
+			(roundrect_rratio 0.243902439)
 			(net 53 "Net-(R3-Pad2)")
 			(pintype "passive")
